Commit message: Marvin can now be simulated in Gazebo
To simulate differential drive control all you need to do is build the catkin workspace and then type the following:
'roslaunch marvin_control test.launch'

File: source/marvin_description/urdf/marvin_dev.urdf (robot description, URDF)
Before this commit: robot marvin, 23 links, 22 joints
Joints:
- joint left_back_caster_to_shoulder: type continuous -> fixed
- joint left_front_caster_to_shoulder: type continuous -> fixed
- joint left_shoulder_horizontal_base: type continuous -> fixed
- joint right_back_caster_to_shoulder: type continuous -> fixed
- joint right_front_caster_to_shoulder: type continuous -> fixed
- joint right_shoulder_horizontal_base: type continuous -> fixed

File: source/marvin_description/urdf/second_marvin.urdf.xacro (robot description, xacro)
@@ -28,9 +28,5 @@
         </inertial>
     </xacro:macro>
-    <gazebo>
-        <plugin name="gazebo_ros_control" filename="libgazebo_ros_control.so">
-            <robotNamespace>/marvin</robotNamespace>
-        </plugin>
-    </gazebo>
+    <xacro:include filename="marvin.gazebo"/>
     <!-- Measurements -->
     <!-- W=Y H=Z D=X -->
@@ -105,5 +101,5 @@
             </collision>
         </link>
-        <joint name="${prefix}_shoulder_horizontal_base" type="continuous">
+        <joint name="${prefix}_shoulder_horizontal_base" type="fixed">
             <origin xyz="
             0.0
@@ -201,5 +197,5 @@
             </collision>
         </link>
-        <joint name="${prefix}_${suffix}_caster_to_shoulder" type="continuous">
+        <joint name="${prefix}_${suffix}_caster_to_shoulder" type="fixed">
             <origin xyz="
                 ${reflect_x * ((shoulder_vertical_x / 2) - (leg_horizontal_x/2))}
@@ -290,22 +286,21 @@
             <axis xyz="0 1 0"/>
         </joint>
-        <!-- Block provides gazbo with info on few additional properties -->
-        <gazebo reference="${prefix}_${suffix}_wheel">
+        <gazebo reference="${prefix}_${suffix}_wheel_link">
             <mu1 value="200.0"/>
             <mu2 value="100.0"/>
-            <kp value="10000000.0" />
+            <kp value="1000000.0" />
             <kd value="1.0" />
-            <material>Gazebo/Black</material>
+            <material>Gazebo/Grey</material>
         </gazebo>
         <!-- This block connects the wheel joint to an actuator (motor), which informs both
         simulation and visualization of the robot -->
         <transmission name="${prefix}_${suffix}_wheel_trans">
-        <type>transmission_interface/SimpleTransmission</type>
-        <actuator name="${prefix}_${suffix}_wheel_motor">
-            <mechanicalReduction>1</mechanicalReduction>
-        </actuator>
-        <joint name="${prefix}_${suffix}_wheel_joint">
-            <hardwareInterface>hardware_interface/VelocityJointInterface</hardwareInterface>
-        </joint>
+            <type>transmission_interface/SimpleTransmission</type>
+            <actuator name="${prefix}_${suffix}_wheel_motor">
+                <mechanicalReduction>1</mechanicalReduction>
+            </actuator>
+            <joint name="${prefix}_${suffix}_wheel_joint">
+                <hardwareInterface>hardware_interface/VelocityJointInterface</hardwareInterface>
+            </joint>
         </transmission>
     </xacro:macro>
