Commit message: Push adjustments to torque

File: source/marvin_description/urdf/marvin_skid.urdf.xacro (robot description, xacro)
@@ -25,5 +25,5 @@
             <origin xyz="0.0 0.0 0.0"/>
             <mass value="${mass}" />
-            <inertia ixx="1.0" ixy="0.0" ixz="0.0" iyy="1.0" iyz="0.0" izz="1.0" />
+            <inertia ixx="0.01" ixy="0.0" ixz="0.0" iyy="0.01" iyz="0.0" izz="0.01" />
         </inertial>
     </xacro:macro>
@@ -35,25 +35,33 @@
     <xacro:property name="shoulder_box_y" value="0.080"/>
     <xacro:property name="shoulder_box_z" value="0.055"/>
+    <xacro:property name="shoulder_box_weight" value="0.050"/>
     <xacro:property name="shoulder_horizontal_x" value="0.040"/>
     <xacro:property name="shoulder_horizontal_y" value="0.085"/>
     <xacro:property name="shoulder_horizontal_z" value="0.020"/>
+    <xacro:property name="shoulder_horizontal_weight" value="0.07241"/>
     <xacro:property name="shoulder_vertical_x" value="0.305"/>
     <xacro:property name="shoulder_vertical_y" value="0.020"/>
     <xacro:property name="shoulder_vertical_z" value="0.060"/>
-    <xacro:property name="leg_horizontal_x" value="0.040"/>
-    <xacro:property name="leg_horizontal_y" value="0.045"/>
-    <xacro:property name="leg_horizontal_z" value="0.020"/>
-    <xacro:property name="leg_vertical_x" value="0.040"/>
-    <xacro:property name="leg_vertical_y" value="0.020"/>
-    <xacro:property name="leg_vertical_z" value="0.110"/>
+    <xacro:property name="shoulder_vertical_weight" value="0.23928"/>
+    <xacro:property name="caster_horizontal_x" value="0.040"/>
+    <xacro:property name="caster_horizontal_y" value="0.045"/>
+    <xacro:property name="caster_horizontal_z" value="0.020"/>
+    <xacro:property name="caster_horizontal_weight" value="0.03834"/>
+    <xacro:property name="caster_vertical_x" value="0.040"/>
+    <xacro:property name="caster_vertical_y" value="0.020"/>
+    <xacro:property name="caster_vertical_z" value="0.110"/>
+    <xacro:property name="caster_vertical_weight" value="0.09371"/>
     <xacro:property name="axle_radius" value="0.015"/>
     <xacro:property name="axle_length" value="0.030"/>
+    <xacro:property name="axle_weight" value="0.160"/>
     <!-- Center of the robot -->
-    <xacro:property name="centre_box_x" value="0.040"/>
-    <xacro:property name="centre_box_y" value="0.100"/>
-    <xacro:property name="centre_box_z" value="0.020"/>
+    <xacro:property name="main_link_x" value="0.040"/>
+    <xacro:property name="main_link_y" value="0.100"/>
+    <xacro:property name="main_link_z" value="0.020"/>
+    <xacro:property name="main_link_weight" value="0.08519"/>
     <!-- Wheel measurements -->
     <xacro:property name="wheel_radius" value="0.055"/>
     <xacro:property name="wheel_length" value="0.050"/>
+    <xacro:property name="wheel_weight" value="0.340"/>
     <!-- Base link -->
     <link name="base_link">
@@ -62,7 +70,7 @@
             <geometry>
                 <box size="
-                    ${centre_box_x}
-                    ${centre_box_y}
-                    ${centre_box_z}"/>
+                    ${main_link_x}
+                    ${main_link_y}
+                    ${main_link_z}"/>
             </geometry>
             <material name="blue"/>
@@ -72,14 +80,14 @@
             <geometry>
                 <box size="
-                    ${centre_box_x}
-                    ${centre_box_y}
-                    ${centre_box_z}"/>
+                    ${main_link_x}
+                    ${main_link_y}
+                    ${main_link_z}"/>
             </geometry>
         </collision>
-        <xacro:default_inertial mass="1"/>
+        <xacro:default_inertial mass="${main_link_weight}"/>
     </link>
     <xacro:macro name="shoulder" params="prefix suffix reflect_y">
         <link name="${prefix}_shoulder_horizontal">
-            <xacro:default_inertial mass="1"/>
+            <xacro:default_inertial mass="${shoulder_horizontal_weight}"/>
             <visual>
                 <origin xyz="0.0 0.0 0.0"/>
@@ -92,5 +100,4 @@
             </visual>
             <collision>
-            <xacro:default_inertial mass="1"/>
                 <origin xyz="0.0 0.0 0.0"/>
                 <geometry>
@@ -104,5 +111,5 @@
             <origin xyz="
             0.0
-            ${reflect_y *((shoulder_horizontal_y / 2) + (centre_box_y / 2))}
+            ${reflect_y *((shoulder_horizontal_y / 2) + (main_link_y / 2))}
             0.0"/>
             <parent link="base_link"/>
@@ -111,5 +118,5 @@
         </joint>
         <link name="${prefix}_shoulder_box">
-            <xacro:default_inertial mass="1"/>
+            <xacro:default_inertial mass="${shoulder_box_weight}"/>
             <visual>
                 <origin xyz="0.0 0.0 0.0"/>
@@ -143,5 +150,5 @@
         </joint>
         <link name="${prefix}_shoulder_vertical">
-            <xacro:default_inertial mass="1"/>
+            <xacro:default_inertial mass="${shoulder_vertical_weight}"/>
             <visual>
                 <origin xyz="0 0.0 0.0" />
@@ -175,12 +182,12 @@
     <xacro:macro name="caster" params="prefix suffix reflect_x reflect_y">
         <link name="${prefix}_${suffix}_caster_horizontal">
-            <xacro:default_inertial mass="1"/>
+            <xacro:default_inertial mass="${caster_horizontal_weight}"/>
             <visual>
                 <origin xyz="0 0.0 0.0" />
                 <geometry>
                     <box size="
-                        ${leg_horizontal_x}
-                        ${leg_horizontal_y}
-                        ${leg_horizontal_z}"/>
+                        ${caster_horizontal_x}
+                        ${caster_horizontal_y}
+                        ${caster_horizontal_z}"/>
                 </geometry>
                 <material name="blue"/>
@@ -190,7 +197,7 @@
                 <geometry>
                     <box size="
-                        ${leg_horizontal_x}
-                        ${leg_horizontal_y}
-                        ${leg_horizontal_z}"/>
+                        ${caster_horizontal_x}
+                        ${caster_horizontal_y}
+                        ${caster_horizontal_z}"/>
                 </geometry>
                 <material name="blue"/>
@@ -199,7 +206,7 @@
         <joint name="${prefix}_${suffix}_caster_to_shoulder" type="fixed">
             <origin xyz="
-                ${reflect_x * ((shoulder_vertical_x / 2) - (leg_horizontal_x/2))}
+                ${reflect_x * ((shoulder_vertical_x / 2) - (caster_horizontal_x/2))}
                 ${reflect_y * (-shoulder_vertical_y /2)}
-                ${-1 * (shoulder_vertical_z / 2 + leg_horizontal_z / 2)}
+                ${-1 * (shoulder_vertical_z / 2 + caster_horizontal_z / 2)}
                 "/>
             <parent link="${prefix}_shoulder_vertical"/>
@@ -208,12 +215,12 @@
         </joint>
         <link name="${prefix}_${suffix}_caster_vertical">
-            <xacro:default_inertial mass="1"/>
-            <visual>
-                <origin xyz="0.0 0.0 0.0"/>
-                <geometry>
-                    <box size="
-                        ${leg_vertical_x}
-                        ${leg_vertical_y}
-                        ${leg_vertical_z}"/>
+            <xacro:default_inertial mass="${caster_vertical_weight}"/>
+            <visual>
+                <origin xyz="0.0 0.0 0.0"/>
+                <geometry>
+                    <box size="
+                        ${caster_vertical_x}
+                        ${caster_vertical_y}
+                        ${caster_vertical_z}"/>
                 </geometry>
                 <material name="green"/>
@@ -223,7 +230,7 @@
                 <geometry>
                     <box size="
-                        ${leg_vertical_x}
-                        ${leg_vertical_y}
-                        ${leg_vertical_z}"/>
+                        ${caster_vertical_x}
+                        ${caster_vertical_y}
+                        ${caster_vertical_z}"/>
                 </geometry>
             </collision>
@@ -232,11 +239,11 @@
             <origin xyz="
                 0
-                ${-reflect_y * (leg_horizontal_y/2 + leg_vertical_y/2)}
-                ${-1 * (leg_vertical_z/2 - leg_horizontal_z/2) }"/>
+                ${-reflect_y * (caster_horizontal_y/2 + caster_vertical_y/2)}
+                ${-1 * (caster_vertical_z/2 - caster_horizontal_z/2) }"/>
             <parent link="${prefix}_${suffix}_caster_horizontal"/>
             <child link="${prefix}_${suffix}_caster_vertical"/>
         </joint>
         <link name="${prefix}_${suffix}_axle">
-            <xacro:default_inertial mass="1"/>
+            <xacro:default_inertial mass="${axle_weight}"/>
             <visual>
                 <origin rpy="${pi/2} 0.0 0.0"/>
@@ -257,5 +264,5 @@
                 0
                 0
-                ${-1 * (leg_vertical_z/2 - axle_radius)}"/>
+                ${-1 * (caster_vertical_z/2 - axle_radius)}"/>
             <parent link="${prefix}_${suffix}_caster_vertical"/>
             <child link="${prefix}_${suffix}_axle"/>
@@ -265,5 +272,5 @@
     <xacro:macro name="wheel" params="prefix suffix reflect_y">
         <link name="${prefix}_${suffix}_wheel_link">
-            <xacro:default_inertial mass="1"/>
+            <xacro:default_inertial mass="${wheel_weight}"/>
             <visual>
                 <origin rpy="${pi/2} 0.0 0.0"/>
@@ -285,9 +292,12 @@
             <child link="${prefix}_${suffix}_wheel_link"/>
             <axis xyz="0 1 0"/>
+            <dynamics damping="1" friction="1" />
         </joint>
         <gazebo reference="${prefix}_${suffix}_wheel_link">
-            <mu1 value="1.0"/>
-            <mu2 value="1.0"/>
-            <kp value="1000000.0" />
+            <mu1 value="2.0"/>
+            <mu2 value="2.0"/>
+            <maxVel value="1"/>
+            <minDepth value="0"/>
+            <kp value="10000.0" />
             <kd value="100.0" />
             <material>Gazebo/Grey</material>
