Commit message: ackermann steering

File: source/marvin_description/urdf/marvin_ackermann.urdf.xacro (robot description, xacro)
@@ -28,5 +28,5 @@
         </inertial>
     </xacro:macro>
-    <xacro:include filename="marvin_skid.gazebo"/>
+    <xacro:include filename="marvin_ackermann.gazebo"/>
     <!-- Measurements -->
     <!-- W=Y H=Z D=X -->
@@ -197,14 +197,29 @@
             </collision>
         </link>
-        <joint name="${prefix}_${suffix}_caster_to_shoulder" type="fixed">
-            <origin xyz="
-                ${reflect_x * ((shoulder_vertical_x / 2) - (leg_horizontal_x/2))}
-                ${reflect_y * (-shoulder_vertical_y /2)}
-                ${-1 * (shoulder_vertical_z / 2 + leg_horizontal_z / 2)}
-                "/>
-            <parent link="${prefix}_shoulder_vertical"/>
-            <child link="${prefix}_${suffix}_caster_horizontal"/>
-            <axis xyz="0 0 1"/>
-        </joint>
+        <xacro:if value="${suffix == 'front'}">
+            <joint name="${prefix}_${suffix}_caster_to_shoulder" type="revolute">
+                <origin xyz="
+                    ${reflect_x * ((shoulder_vertical_x / 2) - (leg_horizontal_x/2))}
+                    ${reflect_y * (-shoulder_vertical_y /2)}
+                    ${-1 * (shoulder_vertical_z / 2 + leg_horizontal_z / 2)}
+                    "/>
+                <parent link="${prefix}_shoulder_vertical"/>
+                <child link="${prefix}_${suffix}_caster_horizontal"/>
+                <axis xyz="0 0 1"/>
+                <limit lower="-1" upper="1" effort="10" velocity="10"/>
+            </joint>
+        </xacro:if>
+        <xacro:if value="${suffix == 'back'}">
+            <joint name="${prefix}_${suffix}_caster_to_shoulder" type="fixed">
+                <origin xyz="
+                    ${reflect_x * ((shoulder_vertical_x / 2) - (leg_horizontal_x/2))}
+                    ${reflect_y * (-shoulder_vertical_y /2)}
+                    ${-1 * (shoulder_vertical_z / 2 + leg_horizontal_z / 2)}
+                    "/>
+                <parent link="${prefix}_shoulder_vertical"/>
+                <child link="${prefix}_${suffix}_caster_horizontal"/>
+                <axis xyz="0 0 1"/>
+            </joint>
+        </xacro:if>
         <link name="${prefix}_${suffix}_caster_vertical">
             <xacro:default_inertial mass="1"/>

Commit message: Updated weights of the ackermann steering robot.
+ updated the steering limits of the wheels.

File: source/marvin_description/urdf/marvin_ackermann.urdf.xacro (robot description, xacro)
@@ -25,5 +25,5 @@
             <origin xyz="0.0 0.0 0.0"/>
             <mass value="${mass}" />
-            <inertia ixx="1.0" ixy="0.0" ixz="0.0" iyy="1.0" iyz="0.0" izz="1.0" />
+            <inertia ixx="0.01" ixy="0.0" ixz="0.0" iyy="0.01" iyz="0.0" izz="0.01" />
         </inertial>
     </xacro:macro>
@@ -35,25 +35,34 @@
     <xacro:property name="shoulder_box_y" value="0.080"/>
     <xacro:property name="shoulder_box_z" value="0.055"/>
+    <xacro:property name="shoulder_box_weight" value="0.050"/>
     <xacro:property name="shoulder_horizontal_x" value="0.040"/>
     <xacro:property name="shoulder_horizontal_y" value="0.085"/>
     <xacro:property name="shoulder_horizontal_z" value="0.020"/>
+    <xacro:property name="shoulder_horizontal_weight" value="0.07241"/>
     <xacro:property name="shoulder_vertical_x" value="0.305"/>
     <xacro:property name="shoulder_vertical_y" value="0.020"/>
     <xacro:property name="shoulder_vertical_z" value="0.060"/>
-    <xacro:property name="leg_horizontal_x" value="0.040"/>
-    <xacro:property name="leg_horizontal_y" value="0.045"/>
-    <xacro:property name="leg_horizontal_z" value="0.020"/>
-    <xacro:property name="leg_vertical_x" value="0.040"/>
-    <xacro:property name="leg_vertical_y" value="0.020"/>
-    <xacro:property name="leg_vertical_z" value="0.110"/>
+    <xacro:property name="shoulder_vertical_weight" value="0.23928"/>
+    <xacro:property name="caster_horizontal_x" value="0.040"/>
+    <xacro:property name="caster_horizontal_y" value="0.045"/>
+    <xacro:property name="caster_horizontal_z" value="0.020"/>
+    <xacro:property name="caster_horizontal_weight" value="0.03834"/>
+    <xacro:property name="caster_vertical_x" value="0.040"/>
+    <xacro:property name="caster_vertical_y" value="0.020"/>
+    <xacro:property name="caster_vertical_z" value="0.110"/>
+    <xacro:property name="caster_vertical_weight" value="0.09371"/>
     <xacro:property name="axle_radius" value="0.015"/>
     <xacro:property name="axle_length" value="0.030"/>
+    <xacro:property name="axle_weight" value="0.160"/>
     <!-- Center of the robot -->
-    <xacro:property name="centre_box_x" value="0.040"/>
-    <xacro:property name="centre_box_y" value="0.100"/>
-    <xacro:property name="centre_box_z" value="0.020"/>
+    <xacro:property name="main_link_x" value="0.040"/>
+    <xacro:property name="main_link_y" value="0.100"/>
+    <xacro:property name="main_link_z" value="0.020"/>
+    <xacro:property name="main_link_weight" value="0.08519"/>
     <!-- Wheel measurements -->
     <xacro:property name="wheel_radius" value="0.055"/>
     <xacro:property name="wheel_length" value="0.050"/>
+    <xacro:property name="wheel_weight" value="0.340"/>
+    <xacro:property name="wheel_turn" value="3.5"/>
     <!-- Base link -->
     <link name="base_link">
@@ -62,7 +71,7 @@
             <geometry>
                 <box size="
-                    ${centre_box_x}
-                    ${centre_box_y}
-                    ${centre_box_z}"/>
+                    ${main_link_x}
+                    ${main_link_y}
+                    ${main_link_z}"/>
             </geometry>
             <material name="blue"/>
@@ -72,14 +81,14 @@
             <geometry>
                 <box size="
-                    ${centre_box_x}
-                    ${centre_box_y}
-                    ${centre_box_z}"/>
+                    ${main_link_x}
+                    ${main_link_y}
+                    ${main_link_z}"/>
             </geometry>
         </collision>
-        <xacro:default_inertial mass="1"/>
+        <xacro:default_inertial mass="${main_link_weight}"/>
     </link>
     <xacro:macro name="shoulder" params="prefix suffix reflect_y">
         <link name="${prefix}_shoulder_horizontal">
-            <xacro:default_inertial mass="1"/>
+            <xacro:default_inertial mass="${shoulder_horizontal_weight}"/>
             <visual>
                 <origin xyz="0.0 0.0 0.0"/>
@@ -92,5 +101,4 @@
             </visual>
             <collision>
-            <xacro:default_inertial mass="1"/>
                 <origin xyz="0.0 0.0 0.0"/>
                 <geometry>
@@ -104,5 +112,5 @@
             <origin xyz="
             0.0
-            ${reflect_y *((shoulder_horizontal_y / 2) + (centre_box_y / 2))}
+            ${reflect_y *((shoulder_horizontal_y / 2) + (main_link_y / 2))}
             0.0"/>
             <parent link="base_link"/>
@@ -111,5 +119,5 @@
         </joint>
         <link name="${prefix}_shoulder_box">
-            <xacro:default_inertial mass="1"/>
+            <xacro:default_inertial mass="${shoulder_box_weight}"/>
             <visual>
                 <origin xyz="0.0 0.0 0.0"/>
@@ -143,5 +151,5 @@
         </joint>
         <link name="${prefix}_shoulder_vertical">
-            <xacro:default_inertial mass="1"/>
+            <xacro:default_inertial mass="${shoulder_vertical_weight}"/>
             <visual>
                 <origin xyz="0 0.0 0.0" />
@@ -175,12 +183,12 @@
     <xacro:macro name="caster" params="prefix suffix reflect_x reflect_y">
         <link name="${prefix}_${suffix}_caster_horizontal">
-            <xacro:default_inertial mass="1"/>
+            <xacro:default_inertial mass="${caster_horizontal_weight}"/>
             <visual>
                 <origin xyz="0 0.0 0.0" />
                 <geometry>
                     <box size="
-                        ${leg_horizontal_x}
-                        ${leg_horizontal_y}
-                        ${leg_horizontal_z}"/>
+                        ${caster_horizontal_x}
+                        ${caster_horizontal_y}
+                        ${caster_horizontal_z}"/>
                 </geometry>
                 <material name="blue"/>
@@ -190,7 +198,7 @@
                 <geometry>
                     <box size="
-                        ${leg_horizontal_x}
-                        ${leg_horizontal_y}
-                        ${leg_horizontal_z}"/>
+                        ${caster_horizontal_x}
+                        ${caster_horizontal_y}
+                        ${caster_horizontal_z}"/>
                 </geometry>
                 <material name="blue"/>
@@ -200,12 +208,12 @@
             <joint name="${prefix}_${suffix}_caster_to_shoulder" type="revolute">
                 <origin xyz="
-                    ${reflect_x * ((shoulder_vertical_x / 2) - (leg_horizontal_x/2))}
+                    ${reflect_x * ((shoulder_vertical_x / 2) - (caster_horizontal_x/2))}
                     ${reflect_y * (-shoulder_vertical_y /2)}
-                    ${-1 * (shoulder_vertical_z / 2 + leg_horizontal_z / 2)}
+                    ${-1 * (shoulder_vertical_z / 2 + caster_horizontal_z / 2)}
                     "/>
                 <parent link="${prefix}_shoulder_vertical"/>
                 <child link="${prefix}_${suffix}_caster_horizontal"/>
                 <axis xyz="0 0 1"/>
-                <limit lower="-1" upper="1" effort="10" velocity="10"/>
+                <limit lower="${-wheel_turn}" upper="${wheel_turn}" effort="10" velocity="10"/>
             </joint>
         </xacro:if>
@@ -213,7 +221,7 @@
             <joint name="${prefix}_${suffix}_caster_to_shoulder" type="fixed">
                 <origin xyz="
-                    ${reflect_x * ((shoulder_vertical_x / 2) - (leg_horizontal_x/2))}
+                    ${reflect_x * ((shoulder_vertical_x / 2) - (caster_horizontal_x/2))}
                     ${reflect_y * (-shoulder_vertical_y /2)}
-                    ${-1 * (shoulder_vertical_z / 2 + leg_horizontal_z / 2)}
+                    ${-1 * (shoulder_vertical_z / 2 + caster_horizontal_z / 2)}
                     "/>
                 <parent link="${prefix}_shoulder_vertical"/>
@@ -223,12 +231,12 @@
         </xacro:if>
         <link name="${prefix}_${suffix}_caster_vertical">
-            <xacro:default_inertial mass="1"/>
-            <visual>
-                <origin xyz="0.0 0.0 0.0"/>
-                <geometry>
-                    <box size="
-                        ${leg_vertical_x}
-                        ${leg_vertical_y}
-                        ${leg_vertical_z}"/>
+            <xacro:default_inertial mass="${caster_vertical_weight}"/>
+            <visual>
+                <origin xyz="0.0 0.0 0.0"/>
+                <geometry>
+                    <box size="
+                        ${caster_vertical_x}
+                        ${caster_vertical_y}
+                        ${caster_vertical_z}"/>
                 </geometry>
                 <material name="green"/>
@@ -238,7 +246,7 @@
                 <geometry>
                     <box size="
-                        ${leg_vertical_x}
-                        ${leg_vertical_y}
-                        ${leg_vertical_z}"/>
+                        ${caster_vertical_x}
+                        ${caster_vertical_y}
+                        ${caster_vertical_z}"/>
                 </geometry>
             </collision>
@@ -247,11 +255,11 @@
             <origin xyz="
                 0
-                ${-reflect_y * (leg_horizontal_y/2 + leg_vertical_y/2)}
-                ${-1 * (leg_vertical_z/2 - leg_horizontal_z/2) }"/>
+                ${-reflect_y * (caster_horizontal_y/2 + caster_vertical_y/2)}
+                ${-1 * (caster_vertical_z/2 - caster_horizontal_z/2) }"/>
             <parent link="${prefix}_${suffix}_caster_horizontal"/>
             <child link="${prefix}_${suffix}_caster_vertical"/>
         </joint>
         <link name="${prefix}_${suffix}_axle">
-            <xacro:default_inertial mass="1"/>
+            <xacro:default_inertial mass="${axle_weight}"/>
             <visual>
                 <origin rpy="${pi/2} 0.0 0.0"/>
@@ -272,5 +280,5 @@
                 0
                 0
-                ${-1 * (leg_vertical_z/2 - axle_radius)}"/>
+                ${-1 * (caster_vertical_z/2 - axle_radius)}"/>
             <parent link="${prefix}_${suffix}_caster_vertical"/>
             <child link="${prefix}_${suffix}_axle"/>
@@ -280,5 +288,5 @@
     <xacro:macro name="wheel" params="prefix suffix reflect_y">
         <link name="${prefix}_${suffix}_wheel_link">
-            <xacro:default_inertial mass="1"/>
+            <xacro:default_inertial mass="${wheel_weight}"/>
             <visual>
                 <origin rpy="${pi/2} 0.0 0.0"/>
@@ -304,5 +312,5 @@
             <mu1 value="1.0"/>
             <mu2 value="1.0"/>
-            <kp value="1000000.0" />
+            <kp value="10000.0" />
             <kd value="100.0" />
             <material>Gazebo/Grey</material>
