Commit message: Test on different machine.

File: source/marvin_description/urdf/chassis.xacro (robot description, xacro)
@@ -43,5 +43,5 @@
       </geometry>
     </collision>
-    <xacro:default_inertial mass="${main_link_weight}" />
+    <!-- <xacro:default_inertial mass="${main_link_weight}" /> -->
   </link>
   <xacro:macro name="shoulder" params="prefix suffix reflect_y">

File: source/marvin_description/urdf/marvin_ackermann.urdf.xacro (robot description, xacro)
@@ -1,5 +1,5 @@
 <?xml version="1.0"?>
 <robot xmlns:xacro="http://www.ros.org/wiki/xacro" name="marvin">
-  <xacro:include filename="marvin_skid.gazebo" />
+  <!-- <xacro:include filename="marvin_skid.gazebo" />-->
   <xacro:include filename="caster_ack.xacro" />
   <xacro:include filename="chassis.xacro" />
@@ -39,9 +39,10 @@
     <xacro:default_inertial mass="0.1" />
   </link>
-  <joint name="middle_front_wheel_joint" type="continuous">
-    <origin xyz="0 0 0" />
+  <joint name="wheel_lead_axle" type="continuous">
+    <origin xyz="0 0 0" rpy="0 0 0"/>
     <parent link="lead_steer" />
     <child link="wheel_lead" />
-    <axis xyz="0 1 0" />
+    <axis xyz="0 1 0"/>
+    <limit effort="1000.0" velocity="0.5"/>
   </joint>
   <!-- Middle back axle test-->
