Commit message: Working ackermann steering.

File: source/marvin_description/urdf/caster.xacro (robot description, xacro)
@@ -54,5 +54,5 @@
       <transmission name="${prefix}_steer_tran">
         <type>transmission_interface/SimpleTransmission</type>
-        <joint name="${prefix}_front_caster_shoulder">
+        <joint name="${prefix}_front_caster_to_shoulder">
           <hardwareInterface>EffortJointInterface</hardwareInterface>
         </joint>

File: source/marvin_description/urdf/caster_ack.xacro (robot description, xacro)
@@ -54,9 +54,9 @@
       <transmission name="${prefix}_steer_tran">
         <type>transmission_interface/SimpleTransmission</type>
-        <joint name="${prefix}_front_caster_shoulder">
-          <hardwareInterface>EffortJointInterface</hardwareInterface>
+        <joint name="${prefix}_front_caster_to_shoulder">
+          <hardwareInterface>hardware_interface/EffortJointInterface</hardwareInterface>
         </joint>
         <actuator name="${prefix}_steer_motor">
-          <hardwareInterface>EffortJointInterface</hardwareInterface>
+          <hardwareInterface>hardware_interface/EffortJointInterface</hardwareInterface>
           <mechanicalReduction>1</mechanicalReduction>
         </actuator>

File: source/marvin_description/urdf/marvin_ackermann.urdf.xacro (robot description, xacro)
@@ -7,4 +7,5 @@
   <xacro:include filename="inertials.xacro" />
   <xacro:include filename="colours.xacro" />
+  <xacro:include filename="marvin_ackermann.gazebo" />
   <!-- Middle front axle test-->
   <link name="front_axle">

File: source/marvin_description/urdf/wheel.xacro (robot description, xacro)
@@ -40,8 +40,8 @@
       <type>transmission_interface/SimpleTransmission</type>
       <joint name="${prefix}_${suffix}_wheel_joint">
-        <hardwareInterface>EffortJointInterface</hardwareInterface>
+        <hardwareInterface>hardware_interface/EffortJointInterface</hardwareInterface>
       </joint>
       <actuator name="${prefix}_${suffix}_motor">
-        <hardwareInterface>EffortJointInterface</hardwareInterface>
+        <hardwareInterface>hardware_interface/EffortJointInterface</hardwareInterface>
         <mechanicalReduction>1</mechanicalReduction>
       </actuator>
