Commit message: Fixed a small mistake in ackermann description

File: src/marvin_description/urdf/marvin_ackermann.urdf.xacro (robot description, xacro)
@@ -217,4 +217,14 @@
                 <limit lower="${-wheel_turn}" upper="${wheel_turn}" effort="10" velocity="10"/>
             </joint>
+            <transmission name="${prefix}_steer_tran">
+                <type>transmission_interface/SimpleTransmission</type>
+                <joint name="${prefix}_front_caster_shoulder">
+                    <hardwareInterface>EffortJointInterface</hardwareInterface>
+                </joint>
+                <actuator name="${prefix}_steer_motor">
+                    <hardwareInterface>EffortJointInterface</hardwareInterface>
+                    <mechanicalReduction>1</mechanicalReduction>
+                </actuator>
+            </transmission>
         </xacro:if>
         <xacro:if value="${suffix == 'back'}">
@@ -284,14 +294,4 @@
             <child link="${prefix}_${suffix}_axle"/>
         </joint>
-        <transmission name="${prefix}_steer_tran">
-            <type>transmission_interface/SimpleTransmission</type>
-            <joint name="${prefix}_front_caster_shoulder">
-                <hardwareInterface>EffortJointInterface</hardwareInterface>
-            </joint>
-            <actuator name="${prefix}_steer_motor">
-                <hardwareInterface>EffortJointInterface</hardwareInterface>
-                <mechanicalReduction>1</mechanicalReduction>
-            </actuator>
-        </transmission>
         <xacro:wheel prefix="${prefix}" suffix="${suffix}" reflect_y="${reflect_y}"/>
     </xacro:macro>
